File: circuts/switch/switch.sch (KiCad schematic (older format))
At the start: 15 parts, among them IC1 ATMEGA328P-TQFP32, IC2 SP3481CN, P1 Power, P2 UART, P3 RS485, P4 CONN_8, P5 CONN_8, U1 LM78L05ACZ, U2 ULN2803L

Commit message: Fixed switch
Parts:
- added P6: BUTTONS, symbol CONN_4
- P4: value CONN_8 -> Relay GND
- P5: value CONN_8 -> Relay 5V
Connections:
- net +12V: now also P5.1 (P1), P5.2 (P2), P5.3 (P3), P5.4 (P4), P5.5 (P5), P5.6 (P6), P5.7 (P7), P5.8 (P8)
- net +5V: no longer P5.1 (P1), P5.2 (P2), P5.3 (P3), P5.4 (P4), P5.5 (P5), P5.6 (P6), P5.7 (P7), P5.8 (P8)
- net GND: now also P6.4 (P4)
- net But2: now reaches IC1.1 ((PCINT19/OC2B/INT1)PD3)
- net But2: now also P6.2 (P2)
- net But1: now reaches IC1.2 ((PCINT20/XCK/T0)PD4)
- net But1: now also P6.1 (P1)
- net Reset: now reaches IC1.29 ((PCINT14/~RESET~)PC6), P2.4 (P4), R2.1
- net But3: now reaches IC1.32 ((PCINT18/INT0)PD2)
- net But3: now also P6.3 (P3)
- no-connect marks 15 -> 12
Changed lines of the file:
@@
 LIBS:valves
 LIBS:asm
-LIBS:automorning-cache
+LIBS:switch-cache
 EELAYER 27 0
 EELAYER END
@@
 	1    0    0    -1
 $EndComp
-NoConn ~ 4300 2050
-NoConn ~ 4200 2050
 NoConn ~ 3700 2050
 NoConn ~ 3600 2050
@@
 NoConn ~ 5300 3750
 NoConn ~ 5300 3600
-NoConn ~ 5300 3200
 $Comp
 L LED D1
@@
 	5750 3300 5750 2950
 Wire Wire Line
-	5850 3100 5850 2950
-Wire Wire Line
 	5350 3500 5350 3050
-Wire Wire Line
-	5350 3050 5950 3050
-Wire Wire Line
-	5950 3050 5950 2950
 Wire Wire Line
 	4200 4950 4200 5300
@@
 Wire Wire Line
 	7300 2900 7300 2850
-$Comp
-L +5V #PWR023
-U 1 1 53B70735
-P 9150 3100
-F 0 "#PWR023" H 9150 3190 20  0001 C CNN
-F 1 "+5V" H 9150 3190 30  0000 C CNN
-F 2 "" H 9150 3100 60  0000 C CNN
-F 3 "" H 9150 3100 60  0000 C CNN
-	1    9150 3100
-	1    0    0    -1
-$EndComp
 Wire Wire Line
 	9150 3100 9150 3300
@@
 P 10200 1850
 F 0 "P4" V 10150 1850 60  0000 C CNN
-F 1 "CONN_8" V 10250 1850 60  0000 C CNN
+F 1 "Relay GND" V 10250 1850 60  0000 C CNN
 F 2 "" H 10200 1850 60  0000 C CNN
 F 3 "" H 10200 1850 60  0000 C CNN
@@
 P 9150 3700
 F 0 "P5" V 9100 3700 60  0000 C CNN
-F 1 "CONN_8" V 9200 3700 60  0000 C CNN
+F 1 "Relay 5V" V 9200 3700 60  0000 C CNN
 F 2 "" H 9150 3700 60  0000 C CNN
 F 3 "" H 9150 3700 60  0000 C CNN
@@
 Wire Wire Line
 	6300 1550 6300 1450
+$Comp
+L +12V #PWR023
+U 1 1 54B154F5
+P 9150 3100
+F 0 "#PWR023" H 9150 3050 20  0001 C CNN
+F 1 "+12V" H 9150 3200 30  0000 C CNN
+F 2 "" H 9150 3100 60  0000 C CNN
+F 3 "" H 9150 3100 60  0000 C CNN
+	1    9150 3100
+	1    0    0    -1
+$EndComp
+Text Label 5350 3050 0    60   ~ 0
+Reset
+Wire Wire Line
+	5350 3050 5950 3050
+Wire Wire Line
+	5950 3050 5950 2950
+Wire Wire Line
+	5850 2950 5850 3100
+$Comp
+L CONN_4 P6
+U 1 1 54B15EA0
+P 5100 1650
+F 0 "P6" V 5050 1650 50  0000 C CNN
+F 1 "BUTTONS" V 5150 1650 50  0000 C CNN
+F 2 "" H 5100 1650 60  0000 C CNN
+F 3 "" H 5100 1650 60  0000 C CNN
+	1    5100 1650
+	0    -1   -1   0
+$EndComp
+$Comp
+L GND #PWR024
+U 1 1 54B15EB9
+P 5250 2100
+F 0 "#PWR024" H 5250 2100 30  0001 C CNN
+F 1 "GND" H 5250 2030 30  0001 C CNN
+F 2 "" H 5250 2100 60  0000 C CNN
+F 3 "" H 5250 2100 60  0000 C CNN
+	1    5250 2100
+	1    0    0    -1
+$EndComp
+Wire Wire Line
+	5250 2100 5250 2000
+Text Label 4200 1900 0    60   ~ 0
+But1
+Text Label 4300 2000 0    60   ~ 0
+But2
+Text Label 5300 2800 0    60   ~ 0
+But3
+Wire Wire Line
+	5300 3200 5300 2250
+Wire Wire Line
+	5300 2250 5150 2250
+Wire Wire Line
+	5150 2250 5150 2000
+Wire Wire Line
+	4300 2050 4400 2050
+Wire Wire Line
+	4400 2050 4400 2150
+Wire Wire Line
+	4400 2150 5050 2150
+Wire Wire Line
+	5050 2150 5050 2000
+Wire Wire Line
+	4200 2050 4200 1900
+Wire Wire Line
+	4200 1900 4800 1900
+Wire Wire Line
+	4800 1900 4800 2100
+Wire Wire Line
+	4800 2100 4950 2100
+Wire Wire Line
+	4950 2100 4950 2000
+Wire Wire Line
+	4300 2000 4300 2050
 $EndSCHEMATC
