File: circuts/switch/switch.kicad_pcb (KiCad board)
At the start: 2 copper layers, 15 parts, among them IC1 ATMEGA328P-TQFP32, IC2 SP3481CN, P1 CONN_2, P2 CONN_4, P3 CONN_2, P4 CONN_8, P5 CONN_8, U1 IRU1015, U2 ULN2803L

Commit message: Fixed switch
Parts:
- added P6: BUTTONS, SIL-4, F.Cu at (52.5, 115.5)
- P1: value CONN_2 -> Power
- P2: value CONN_4 -> UART
- P3: value CONN_2 -> RS485
- P4: value CONN_8 -> Relay GND
- P5: value CONN_8 -> Relay 5V
- U1: value IRU1015 -> LM78L05ACZ; moved to B.Cu
- moved P1 76.3 mm to (26.2, 115.3), turned to 0 degrees
- moved R4 65.9 mm to (50.9, 120.6)
- moved R2 63.8 mm to (36.1, 118.2), turned to 0 degrees
- moved U1 62.9 mm to (26.2, 120.3)
- moved R5 57.4 mm to (50.6, 133.2)
- moved P3 57.2 mm to (55.9, 126.3)
- moved IC2 57.1 mm to (50.6, 126.3)
- moved R3 56.3 mm to (45.9, 132.0), turned to 90 degrees
- moved IC1 56.0 mm to (39.7, 125.8)
- moved D1 55.3 mm to (40.1, 132.9), turned to 180 degrees
- moved U2 53.3 mm to (26.0, 123.6)
- moved R1 53.2 mm to (33.0, 132.4)
- moved P4 53.2 mm to (17.4, 124.6)
- moved P5 49.6 mm to (14.8, 124.6), turned to 270 degrees
- moved P2 42.8 mm to (39.5, 115.4), turned to 180 degrees
Connections:
- IC1 pad 1: (no net) -> /But2
- IC1 pad 2: (no net) -> /But1
- IC1 pad 29: N-0000017 (its old number) -> /Reset
- IC1 pad 32: (no net) -> /But3
- P2 pad 4: N-0000017 (its old number) -> /Reset
- P5 pad 1: +5V -> +12V
- P5 pad 2: +5V -> +12V
- P5 pad 3: +5V -> +12V
- P5 pad 4: +5V -> +12V
- P5 pad 5: +5V -> +12V
- P5 pad 6: +5V -> +12V
- P5 pad 7: +5V -> +12V
- P5 pad 8: +5V -> +12V
- R2 pad 1: N-0000017 (its old number) -> /Reset
- U1 pad 1: GND -> +12V
- U1 pad 2: +5V -> GND
- U1 pad 3: +12V -> +5V
Routing:
- net GND: track 0.00 -> 105.7 mm, vias 0 -> 1
- net +5V: track 0.00 -> 51.0 mm, vias 0 -> 4
- net +12V: track 0.00 -> 36.2 mm, vias 0 -> 5
- net /DI: track 0.00 -> 22.4 mm, vias 0 -> 2
- net /DO: track 0.00 -> 19.3 mm
- net /Reset: track 0.00 -> 18.0 mm
- net /Dir: track 0.00 -> 12.8 mm
- net /But3: track 0.00 -> 12.7 mm, vias 0 -> 1
- net /But2: track 0.00 -> 11.0 mm, vias 0 -> 1
- net N-0000017: track 0.00 -> 10.9 mm
- net /But1: track 0.00 -> 10.2 mm, vias 0 -> 1
- net N-0000021: track 0.00 -> 9.05 mm
- net N-000009: track 0.00 -> 6.73 mm
- net N-0000013: track 0.00 -> 6.55 mm
- net N-0000020: track 0.00 -> 6.25 mm
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Other:
- board outline added: 45.4 x 50 mm
- board text added: "+12 -"
- board text added: "B1 B2 B3 G"
- board text added: "R G I O"
- board text added: "RELAY"
- board text added: "RS485"
- board text added: "SH Switch v1.0 2015"

Commit message: Sended to prodaction
Parts:
- added D1: LED, LED-0805, F.Cu at (27.0, 43.0)
- added IC1: ATMEGA328P-TQFP32, TQFP32, F.Cu at (26.6, 35.9)
- added IC2: SP3481CN, so-8, F.Cu at (37.5, 36.4)
- added P1: Power, C2, F.Cu at (13.1, 25.4)
- added P2: UART, SIL-4, F.Cu at (26.4, 25.5)
- added P3: RS485, C2, F.Cu at (42.8, 36.4)
- added P4: Relay GND, SIL-8, F.Cu at (4.30, 34.7)
- added P5: Relay 5V, SIL-8, F.Cu at (1.70, 34.7)
- added P6: BUTTONS, SIL-4, F.Cu at (39.4, 25.6)
- added R1: 1K, SM1206, F.Cu at (19.9, 42.5)
- added R2: 1K, SM1206, F.Cu at (23.0, 28.3)
- added R3: 10K, SM1206, F.Cu at (32.8, 42.1)
- added R4: 560, SM1206, F.Cu at (37.8, 30.7)
- added R5: 560, SM1206, F.Cu at (37.5, 43.3)
- added U1: LM78L05ACZ, DPAK3, B.Cu at (13.1, 30.4)
- added U2: ULN2803L, SO18L, F.Cu at (12.9, 33.7)
- moved D1 113.5 mm to (27.0, 20.2)
- moved IC1 113.5 mm to (26.6, 13.1)
- moved IC2 113.5 mm to (37.5, 13.6)
- moved P1 113.5 mm to (13.1, 2.60)
- moved P2 113.5 mm to (26.4, 2.70)
- moved P3 113.5 mm to (42.8, 13.6)
- moved P6 113.5 mm to (39.4, 2.80)
- moved R1 113.5 mm to (19.9, 19.7)
- moved R2 113.5 mm to (23.0, 5.50)
- moved R3 113.5 mm to (32.8, 19.3)
- moved U1 113.5 mm to (13.1, 7.60)
- moved P4 113.5 mm to (4.30, 11.9)
- moved P5 113.5 mm to (1.70, 11.9)
- moved R4 113.5 mm to (37.8, 7.90)
- moved R5 113.5 mm to (37.5, 20.5)
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Routing:
- net GND: track 105.7 -> 211.4 mm, vias 1 -> 2
- net +5V: track 51.0 -> 102.0 mm, vias 4 -> 8
- net +12V: track 36.2 -> 72.5 mm, vias 5 -> 10
- net /DI: track 22.4 -> 44.8 mm, vias 2 -> 4
- net /DO: track 19.3 -> 38.6 mm
- net /Reset: track 18.0 -> 36.0 mm
- net /Dir: track 12.8 -> 25.6 mm
- net /But3: track 12.7 -> 25.4 mm, vias 1 -> 2
- net /But2: track 11.0 -> 22.0 mm, vias 1 -> 2
- net N-0000017: track 10.9 -> 21.8 mm
- net /But1: track 10.2 -> 20.3 mm, vias 1 -> 2
- net N-0000021: track 9.05 -> 18.1 mm
- net N-000009: track 6.73 -> 13.5 mm
- net N-0000013: track 6.55 -> 13.1 mm
- net N-0000020: track 6.25 -> 12.5 mm
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Other:
- board size 45.4 x 50 mm -> 45.5 x 45.1 mm
